File: LampaPass-STD-Board/Battery_Charging_Module.kicad_sch (KiCad schematic)
At the start: 0 parts

Commit message: Added a draft version of the battery protection and charge scheme. Updated Main IC list.
Parts:
- added C1: 100nF, Resistor_SMD:R_0402_1005Metric, symbol Device:C
- added C2: 0.47uF, Resistor_SMD:R_0402_1005Metric, symbol Device:C
- added C3, C4: 4.7u, Capacitor_SMD:C_1206_3216Metric, symbol Device:C_Polarized_US
- added J2: Termistor, symbol Connector_Generic:Conn_01x02
- added J2: Batt_conn, symbol Connector_Generic:Conn_01x02
- added Q1: FDS6898A, Package_SO:SOIC-8_3.9x4.9mm_P1.27mm, symbol Transistor_FET:FDS6898A
- added Q2: Q_PMOS_GDS, symbol Device:Q_PMOS_GDS
- added R1: 330, Resistor_SMD:R_0402_1005Metric, symbol Device:R
- added R2: 2.7K, Resistor_SMD:R_0402_1005Metric, symbol Device:R
- added R3: 100K, Resistor_SMD:R_0402_1005Metric, symbol Device:R
- added R4: 1.1, Resistor_SMD:R_0402_1005Metric, symbol Device:R
- added R5: 10K, Resistor_SMD:R_0402_1005Metric, symbol Device:R
- added R6: 15K, Resistor_SMD:R_0402_1005Metric, symbol Device:R
- added U1: MCP73841-410I/UN, Package_SO:MSOP-10_3x3mm_P0.5mm, symbol LampaPass_Power_Management:MCP73841-410I/UN
- added U2: AP9101CK6, Package_TO_SOT_SMD:SOT-23-6, symbol LampaPass_Power_Management:AP9101CK6
Connections:
- new net: C2.1, U1.7 (TIMER)
- new net: R2.1, U2.2 (VM)
- new net: J2.1 (Pin_1), R5.2, R6.2, U1.6 (THERM)
- new net: R3.2, U1.4 (EN)
- new net: Q2.1 (G), U1.10 (DRV)
- new net: Q2.3 (S), R4.2, U1.1 (Sense)
- new net: R5.1, U1.5 (THREF)
- new net: C1.1, J2.2 (Pin_2), Q1.1 (S1), U2.6 (VSS)
- new net: Q1.2 (G1), U2.1 (DO)
- new net: Q1.5 (D2), Q1.6 (D2), Q1.7 (D1), Q1.8 (D1)
- new net: C1.2, R1.2, U2.5 (VDD)
- new net: Q1.4 (G2), U2.3 (CO)
- new net +9V: C4.1, R4.1, U1.2 (VDD)
- new net Charge_EN: R3.1
- new net Charge_info: U1.3 (STAT1)
- new net GND: C2.2, C3.2, C4.2, J2.2 (Pin_2), Q1.3 (S2), R2.2, R6.1, U1.8 (VSS)
- new net VDD: C3.1, J2.1 (Pin_1), Q2.2 (D), R1.1, U1.9 (VBAT)
Other:
- note added: "+"
- note added: "-"
